File: KicadProject/NXP_DMX.sch (KiCad schematic (older format))
At the start: 56 parts, among them J1 USB, J2 Debug_Header, J3 4_Pos, J4 XLR, Q1 BJT_PNP, SW1 Button, SW2 Button, U1 LPC11U14, U2 ZLDO1117, U3 1G_NAND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

Commit message: Add label to schematic
Other:
- note added: "Isolated NXP AN11154 by EmbeddedEE"
Changed lines of the file:
@@
 	10200 5500 10350 5500
 Connection ~ 10350 5500
+Text Notes 6700 7750 0    60   ~ 0
+Isolated NXP AN11154 by EmbeddedEE
 $EndSCHEMATC
